File: microprocessor.kicad_sch (KiCad schematic)
At the start: 18 parts, among them J1 Conn_ARM_JTAG_SWD_10, J4 Conn_01x04, U7 STM32F030F4Px

Commit message: cleanup rev-a
Parts:
- added C25: 100n, Capacitor_SMD:C_0603_1608Metric, symbol Device:C_Small
- added R51 (x2): 1k, Resistor_SMD:R_0603_1608Metric, symbol Device:R_Small
- added U6: 74LVC2G14, Package_TO_SOT_SMD:SOT-23-6, symbol 74xGxx:74LVC2G14
Connections:
- net +3.3V: now also R51.1, R51.1
- net GND: now also C25.2, U6.2 (GND), U6.2 (GND)
- net SW_NEG: now also U6.4; no longer TP6.1, U7.13 (PA7)
- net SW_POS: now also U6.6; no longer TP6.1, U7.12 (PA6)
- new net +5V: C25.1, U6.5 (VCC), U6.5 (VCC)
- new net SW_NEG_3v3: R51.2, TP6.1, U6.3, U7.13 (PA7)
- new net SW_POS_3v3: R51.2, TP6.1, U6.1, U7.12 (PA6)
Other:
- note added: "4066 has VinH_min of >3.3V, so we need 5V swing"

Commit message: Notes during bringup of rev. a.
Parts:
- R51: value 1k -> dnp
- R51: value 1k -> 51k
Other:
- note added: "BOOT0=L"
Changed lines of the file:
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@@
     (stroke (width 0) (type default))
+  )
+  (polyline (pts (xy 128.27 48.26) (xy 138.43 48.26))
+    (stroke (width 0) (type dash))
   )
   (wire (pts (xy 71.12 60.96) (xy 71.12 62.23))
@@
     (stroke (width 0) (type default))
   )
+  (polyline (pts (xy 128.27 36.83) (xy 138.43 36.83))
+    (stroke (width 0) (type dash))
+  )
   (wire (pts (xy 137.16 38.1) (xy 137.16 39.37))
     (stroke (width 0) (type default))
@@
     (stroke (width 0) (type default))
   )
+  (polyline (pts (xy 128.27 36.83) (xy 128.27 48.26))
+    (stroke (width 0) (type dash))
+  )
   (wire (pts (xy 138.43 62.23) (xy 127 62.23))
     (stroke (width 0) (type default))
@@
     (stroke (width 0) (type default))
   )
+  (polyline (pts (xy 138.43 36.83) (xy 138.43 48.26))
+    (stroke (width 0) (type dash))
+  )
   (wire (pts (xy 137.16 39.37) (xy 138.43 39.37))
     (stroke (width 0) (type default))
@@
   )
   (text "TIM3_CH2" (at 185.42 53.34 0)
+    (effects (font (size 1.27 1.27)) (justify left bottom))
+  )
+  (text "BOOT0=L" (at 128.27 48.26 0)
     (effects (font (size 1.27 1.27)) (justify left bottom))
   )
@@
   (global_label "SW_NEG" (shape input) (at 238.76 93.98 0) (fields_autoplaced)
     (effects (font (size 1.27 1.27)) (justify left))
-    (property "Intersheetrefs" "${INTERSHEET_REFS}" (at 249.1232 93.98 0)
-      (effects (font (size 1.27 1.27)) (justify left) hide)
-    )
     (property "Intersheetrefs" "${INTERSHEET_REFS}" (at 238.76 96.1708 0)
       (effects (font (size 1.27 1.27)) (justify left) hide)
     )
-    (property "Intersheetrefs" "${INTERSHEET_REFS}" (at 238.76 96.1708 0)
-      (effects (font (size 1.27 1.27)) (justify left) hide)
-    )
-    (property "Intersheetrefs" "${INTERSHEET_REFS}" (at 238.76 96.1708 0)
-      (effects (font (size 1.27 1.27)) (justify left) hide)
-    )
   )
   (global_label "SW_POS" (shape input) (at 238.76 80.01 0) (fields_autoplaced)
     (effects (font (size 1.27 1.27)) (justify left))
-    (property "Intersheetrefs" "${INTERSHEET_REFS}" (at 249.1837 80.01 0)
-      (effects (font (size 1.27 1.27)) (justify left) hide)
-    )
-    (property "Intersheetrefs" "${INTERSHEET_REFS}" (at 238.76 82.2008 0)
-      (effects (font (size 1.27 1.27)) (justify left) hide)
-    )
     (property "Intersheetrefs" "${INTERSHEET_REFS}" (at 238.76 83.8518 0)
       (effects (font (size 1.27 1.27)) (justify left) hide)
@@
   (global_label "RESOLVER_TX" (shape input) (at 212.09 29.21 0) (fields_autoplaced)
     (effects (font (size 1.27 1.27)) (justify left))
-    (property "Intersheetrefs" "${INTERSHEET_REFS}" (at 36.83 -25.4 0)
-      (effects (font (size 1.27 1.27)) hide)
-    )
     (property "Intersheetrefs" "${INTERSHEET_REFS}" (at 227.7146 29.21 0)
       (effects (font (size 1.27 1.27)) (justify left) hide)
@@
       (effects (font (size 1.27 1.27)))
     )
-    (property "Value" "1k" (at 134.62 43.18 90)
+    (property "Value" "dnp" (at 134.62 43.18 90)
       (effects (font (size 1.27 1.27)))
     )
@@
       (effects (font (size 1.27 1.27)))
     )
-    (property "Value" "1k" (at 222.25 68.58 0)
+    (property "Value" "51k" (at 222.25 68.58 0)
       (effects (font (size 1.27 1.27)))
     )
@@
       (effects (font (size 1.27 1.27)))
     )
-    (property "Value" "1k" (at 134.62 45.72 90)
+    (property "Value" "51k" (at 134.62 45.72 90)
       (effects (font (size 1.27 1.27)))
     )
@@
       (effects (font (size 1.27 1.27)))
     )
-    (property "Value" "1k" (at 215.9 68.58 0)
+    (property "Value" "51k" (at 215.9 68.58 0)
       (effects (font (size 1.27 1.27)))
     )
@@
       (effects (font (size 1.27 1.27)))
     )
-    (property "Value" "1k" (at 130.81 27.94 0)
-      (effects (font (size 1.27 1.27)))
-    )
+    (property "Value" "51k" (at 130.81 27.94 0)
+      (effects (font (size 1.27 1.27)))
+    )
