File: resolver-to-sincos.kicad_pcb (KiCad board)
At the start: 4 copper layers, 75 x 75 mm, 135 parts, among them J1 Conn_ARM_JTAG_SWD_10, J2 Screw_Terminal_01x08, J3 Screw_Terminal_01x08, J4 Conn_01x04, U1 LM4040DBZ-2.5, U2 MCP6484, U3 4066, U4 MCP6484, U5 MCP6484, U7 STM32F030F4Px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

Commit message: cleanup rev-a
Parts:
- added C35: 100n, Capacitor_SMD:C_0603_1608Metric, F.Cu at (146.3, 132.6)
- added R64: 1k, Resistor_SMD:R_0603_1608Metric, F.Cu at (143.8, 127.7)
- added R65: 1k, Resistor_SMD:R_0603_1608Metric, F.Cu at (147.8, 125.2)
- added U6: 74LVC2G14, Package_TO_SOT_SMD:SOT-23-6, F.Cu at (146.3, 129.5)
Connections:
- TP10 pad 1: SW_POS -> /Microprocessor/SW_POS_3v3
- TP11 pad 1: SW_NEG -> /Microprocessor/SW_NEG_3v3
- U7 pad 12: SW_POS -> /Microprocessor/SW_POS_3v3
- U7 pad 13: SW_NEG -> /Microprocessor/SW_NEG_3v3
Routing:
- net SW_POS: track 73.9 -> 19.3 mm
- net /Microprocessor/SW_POS_3v3: track 0.00 -> 53.2 mm
- net SW_NEG: track 71.4 -> 20.2 mm
- net /Microprocessor/SW_NEG_3v3: track 0.00 -> 50.0 mm
- net +3.3V: track 193.7 -> 212.1 mm, vias 6 -> 8
- net +5V: track 33.0 -> 36.6 mm, vias 13 -> 14
- net GND: track 57.7 -> 58.4 mm, vias 45 -> 47
- net Net-(U7-PA9): track 6.99 -> 6.33 mm
Other:
- board text added: "1,2 → +5V Supply 3,4 → COS P,N 5,6 → SIN P,N 7,8 → ⏚"
- board text added: "cos n"
- board text added: "cos p"
- board text added: "resolver-to-sincos rev A vogelchr@vogel.cx https://github.com/vogelchr/"
- board text added: "sin n"
- board text added: "sin p"
- board text added: "tx n"
- board text added: "tx p"
- board text removed: "1,2 → ⏚ 3,4 → COS P,N 5,6 → SIN P,N 7,8 → +5V Supply"

Commit message: reva - small tweaks
Other:
- board text added: "resolver-to-sincos rev A 2022/12 vogelchr@vogel.cx"
- board text removed: "resolver-to-sincos rev A vogelchr@vogel.cx https://github.com/vogelchr/"
Changed lines of the file:
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@@
     (effects (font (size 1.5 1.5) (thickness 0.3) bold) (justify left bottom mirror))
-  )
-  (gr_text "resolver-to-sincos rev A\nvogelchr@vogel.cx\nhttps://github.com/vogelchr/" (at 173.736 159.512) (layer "B.Cu")
-    (effects (font (size 1.5 1.5) (thickness 0.25) bold) (justify left bottom mirror))
   )
   (gr_text "GND" (at 122.936 102.108 90) (layer "B.Cu")
@@
     (effects (font (size 1.2 1.2) (thickness 0.15)) (justify left bottom))
   )
+  (gr_text "resolver-to-sincos\nrev A 2022/12\nvogelchr@vogel.cx" (at 162.052 130.048) (layer "F.SilkS")
+    (effects (font (size 0.75 0.75) (thickness 0.15) bold) (justify left bottom))
+  )
   (gr_text "pa4" (at 123.952 124.968) (layer "F.SilkS")

Commit message: Notes during bringup of rev. a.
Parts:
- C1, C10, C11, C12, C13, C17, C19, C2, C20, C3, C4, C5, C6, C7, C8, C9: value 1n0 -> 0.1n
- C15, C16, C21, C22: value 1n0 -> 10n
- R15, R16, R17, R18, R19, R20, R21, R22: value 1k -> 68R
- R2, R23, R24, R27, R28, R3, R31, R36, R37, R4, R40, R41, R42, R49, R5, R51, R52, R53, R54, R61, R62, R63: value 1k -> 27k
- R25, R26, R29, R30, R38, R39, R43, R44, R56, R57, R58, R64, R65: value 1k -> 51k
- R32, R33, R34, R35, R45, R46, R47, R48: value 1k -> 33k
- R50, R59: value 2k -> 51k
- R6, R7: value 27R -> 68R
