File: resolver-to-sincos.kicad_sch (KiCad schematic)
At the start: 110 parts, among them J2 Screw_Terminal_01x08, J3 Screw_Terminal_01x08, U1 LM4040DBZ-2.5, U2 MCP6484, U3 4066, U4 MCP6484, U5 MCP6484, U8 AP1117-33

Commit message: cleanup rev-a
Parts:
- added R61, R62, R63: 1k, Resistor_SMD:R_0603_1608Metric, symbol Device:R_Small
- added TP18, TP19, TP20, TP21: TestPoint, TestPoint:TestPoint_Pad_1.5x1.5mm, symbol Connector:TestPoint
Connections:
- net +3.3V: now also TP18.1
- net U_REF: now also R63.1; no longer U5.12 (+)
- net at U5.13 (-): now also R61.1, R62.2; no longer U5.14
- new net: R63.2, TP21.1, U5.12 (+)
- new net: R61.2, TP19.1, U5.14
- new net: R62.1, TP20.1
- no-connect marks 1 -> 0
Other:
- moved on the sheet: TP8, TP9, U5D

Commit message: Notes during bringup of rev. a.
Parts:
- C1, C10, C11, C12, C13, C17, C19, C2, C20, C3, C4, C5, C6, C7, C8, C9: value 1n0 -> 0.1n
- C15, C16, C21, C22: value 1n0 -> 10n
- R15, R16, R17, R18, R19, R20, R21, R22: value 1k -> 68R
- R2, R23, R24, R27, R28, R3, R31, R36, R37, R4, R40, R41, R42, R49, R5, R51, R52, R53, R54, R61, R62, R63: value 1k -> 27k
- R25, R26, R29, R30, R38, R39, R43, R44: value 1k -> 51k
- R32, R33, R34, R35, R45, R46, R47, R48: value 1k -> 33k
- R50, R59: value 2k -> 51k
- R6, R7: value 27R -> 68R
Other:
- note added: "27k in front of ESD protection"
- note added: "Sallen Key 2nd Order LP 500 Hz"
- note added: "Z+ = Z- = 20.5kOhm, C=0.1nF: f=77.6kHz"
- note added: "gain +/- 1, fLP = 77.6kHz"
- note added: "gain diff. input to output = 1"
